Commit message: matt first commmt

File: launch/ego_racecar_backup.xacro (robot description, xacro)
@@ -18,5 +18,5 @@
     <color rgba="0.3 0.57 1. 1."/>
   </material>
-  <link name="base_link">
+  <link name="${car_name}/base_link">
     <visual>
       <origin xyz="${wheelbase/2} 0 ${ground_offset+height/2}"/>
@@ -28,9 +28,9 @@
   </link>
   <joint name="base_to_laser_model" type="fixed">
-    <parent link="base_link"/>
-    <child link="laser_model"/>
+    <parent link="${car_name}/base_link"/>
+    <child link="${car_name}/laser_model"/>
     <origin xyz="${laser_distance_from_base_link} 0 ${ground_offset+height+(laser_height/2)}"/>
   </joint>
-  <link name="laser_model">
+  <link name="${car_name}/laser_model">
     <visual>
       <geometry>
@@ -41,9 +41,9 @@
   </link>
   <joint name="$base_to_back_left_wheel" type="fixed">
-    <parent link="base_link"/>
-    <child link="back_left_wheel"/>
+    <parent link="${car_name}/base_link"/>
+    <child link="${car_name}/back_left_wheel"/>
     <origin xyz="0 ${(wheel_length+width)/2} ${wheel_radius}"/>
   </joint>
-  <link name="back_left_wheel">
+  <link name="${car_name}/back_left_wheel">
     <visual>
       <geometry>
@@ -55,9 +55,9 @@
   </link>
   <joint name="base_to_back_right_wheel" type="fixed">
-    <parent link="base_link"/>
-    <child link="back_right_wheel"/>
+    <parent link="${car_name}/base_link"/>
+    <child link="${car_name}/back_right_wheel"/>
     <origin xyz="0 ${-(wheel_length+width)/2} ${wheel_radius}"/>
   </joint>
-  <link name="back_right_wheel">
+  <link name="${car_name}/back_right_wheel">
     <visual>
       <geometry>
@@ -69,14 +69,14 @@
   </link>
   <joint name="base_to_front_left_hinge" type="fixed">
-    <parent link="base_link"/>
-    <child link="front_left_hinge"/>
+    <parent link="${car_name}/base_link"/>
+    <child link="${car_name}/front_left_hinge"/>
     <origin xyz="${wheelbase} ${(wheel_length+width)/2} ${wheel_radius}"/>
   </joint>
-  <link name="front_left_hinge"/>
+  <link name="${car_name}/front_left_hinge"/>
   <joint name="front_left_hinge_to_wheel" type="continuous">
-    <parent link="front_left_hinge"/>
-    <child link="front_left_wheel"/>
+    <parent link="${car_name}/front_left_hinge"/>
+    <child link="${car_name}/front_left_wheel"/>
   </joint>
-  <link name="front_left_wheel">
+  <link name="${car_name}/front_left_wheel">
     <visual>
       <geometry>
@@ -88,14 +88,14 @@
   </link>
   <joint name="base_to_front_right_hinge" type="fixed">
-    <parent link="base_link"/>
-    <child link="front_right_hinge"/>
+    <parent link="${car_name}/base_link"/>
+    <child link="${car_name}/front_right_hinge"/>
     <origin xyz="${wheelbase} ${-(wheel_length+width)/2} ${wheel_radius}"/>
   </joint>
-  <link name="front_right_hinge"/>
+  <link name="${car_name}/front_right_hinge"/>
   <joint name="front_right_hinge_to_wheel" type="continuous">
-    <parent link="front_right_hinge"/>
-    <child link="front_right_wheel"/>
+    <parent link="${car_name}/front_right_hinge"/>
+    <child link="${car_name}/front_right_wheel"/>
   </joint>
-  <link name="front_right_wheel">
+  <link name="${car_name}/front_right_wheel">
     <visual>
       <geometry>
