Commit message: lots of testing done, still need to do pose error calculations

File: launch/ego_racecar.xacro (robot description, xacro)
@@ -2,5 +2,5 @@
 <!-- A simple model of the racecar for rviz -->
 <robot xmlns:xacro="http://www.ros.org/wiki/xacro" name="racecar">
-  <xacro:property name="wheelbase" value="0.3302" />
+  <xacro:property name="wheelbase" value="0.324" />
   <xacro:property name="width" value="0.2032" />
   <xacro:property name="height" value="0.1" />
